File: ESP32_Playboard.sch (KiCad schematic (older format))
At the start: 40 parts, among them J1 USB_B_Micro, J2 TF_PUSH, Q1 Q_NPN_BEC, Q2 Q_NPN_BEC, Q3 Q_NPN_BEC, SW1 SW_SPST, SW2 SW_SPST, U1 AMS1117-3.3, U2 USBLC6-2SC6, U3 CH340G, U4 ESP32-WROVER-I, U5 MPU-6050, U6 SHT30-DIS, Y1 12MHz

Commit message: Finished basic PCB layout (no routing)
Parts:
- D1: footprint PlayboardLib:LED_SMD-4 -> PlayboardLib:LED-SMD-4
Connections:
- net GND: now also D2.1 (K); no longer R4.1
- net at R4.2: now also Q1.2 (E); no longer D2.1 (K)
- net at D2.2 (A): now also R4.1; no longer Q1.2 (E)
Other:
- moved on the sheet: D2, R4
Changed lines of the file:
@@
 F 0 "D1" H 7800 3165 50  0000 C CNN
 F 1 "IRM-H638T_TR2" H 7800 3074 50  0000 C CNN
-F 2 "PlayboardLib:LED_SMD-4" H 7550 3000 50  0001 C CNN
+F 2 "PlayboardLib:LED-SMD-4" H 7550 3000 50  0001 C CNN
 F 3 "" H 7550 3000 50  0001 C CNN
 F 4 "https://www.lcsc.com/product-detail/C91447.html" H 7550 3000 50  0001 C CNN "LCSC Link"
@@
 L Device:R_Small R4
 U 1 1 629BDA54
-P 9600 3400
-F 0 "R4" V 9450 3550 50  0000 C CNN
-F 1 "47" V 9550 3550 50  0000 C CNN
-F 2 "Resistor_SMD:R_0603_1608Metric" H 9600 3400 50  0001 C CNN
-F 3 "~" H 9600 3400 50  0001 C CNN
-F 4 "https://www.lcsc.com/product-detail/C1211.html" H 9600 3400 50  0001 C CNN "LCSC Link"
-F 5 "C1211" H 9600 3400 50  0001 C CNN "LCSC Part Number"
-F 6 "UNI-ROYAL(Uniroyal Elec)" H 9600 3400 50  0001 C CNN "Manufacturer"
-F 7 "0603WAJ0470T5E" H 9600 3400 50  0001 C CNN "Manufacturer Part Number"
-	1    9600 3400
+P 9350 3400
+F 0 "R4" V 9200 3550 50  0000 C CNN
+F 1 "47" V 9300 3550 50  0000 C CNN
+F 2 "Resistor_SMD:R_0603_1608Metric" H 9350 3400 50  0001 C CNN
+F 3 "~" H 9350 3400 50  0001 C CNN
+F 4 "https://www.lcsc.com/product-detail/C1211.html" H 9350 3400 50  0001 C CNN "LCSC Link"
+F 5 "C1211" H 9350 3400 50  0001 C CNN "LCSC Part Number"
+F 6 "UNI-ROYAL(Uniroyal Elec)" H 9350 3400 50  0001 C CNN "Manufacturer"
+F 7 "0603WAJ0470T5E" H 9350 3400 50  0001 C CNN "Manufacturer Part Number"
+	1    9350 3400
 	0    1    1    0
 $EndComp
@@
 L Device:LED_Small D2
 U 1 1 629B2955
-P 9350 3400
-F 0 "D2" H 9450 3450 50  0000 C CNN
-F 1 "IR LED" H 9450 3550 50  0000 C CNN
-F 2 "LED_SMD:LED_0603_1608Metric" V 9350 3400 50  0001 C CNN
-F 3 "~" V 9350 3400 50  0001 C CNN
-F 4 "https://www.lcsc.com/product-detail/C50494.html" H 9350 3400 50  0001 C CNN "LCSC Link"
-F 5 "C50494" H 9350 3400 50  0001 C CNN "LCSC Part Number"
-F 6 "Everlight Elec" H 9350 3400 50  0001 C CNN "Manufacturer"
-F 7 "MIR60363T" H 9350 3400 50  0001 C CNN "Manufacturer Part Number"
-	1    9350 3400
+P 9600 3400
+F 0 "D2" H 9700 3450 50  0000 C CNN
+F 1 "IR LED" H 9700 3550 50  0000 C CNN
+F 2 "LED_SMD:LED_0603_1608Metric" V 9600 3400 50  0001 C CNN
+F 3 "~" V 9600 3400 50  0001 C CNN
+F 4 "https://www.lcsc.com/product-detail/C50494.html" H 9600 3400 50  0001 C CNN "LCSC Link"
+F 5 "C50494" H 9600 3400 50  0001 C CNN "LCSC Part Number"
+F 6 "Everlight Elec" H 9600 3400 50  0001 C CNN "Manufacturer"
+F 7 "MIR60363T" H 9600 3400 50  0001 C CNN "Manufacturer Part Number"
+	1    9600 3400
 	-1   0    0    1
 $EndComp
@@
 NoConn ~ 4750 4500
 NoConn ~ 4750 4700
+NoConn ~ 4750 4900
+NoConn ~ 4750 5000
+NoConn ~ 3550 5900
+Text Label 3100 4600 0    50   ~ 0
+GPIO0
+Wire Wire Line
+	4750 4800 5200 4800
+Wire Wire Line
+	4750 4600 5200 4600
+Text Label 5200 4800 2    50   ~ 0
+IR_SEND
+Text Label 5200 4600 2    50   ~ 0
+IR_RECV
+$Comp
+L power:GND #PWR020
+U 1 1 61CED5C0
+P 4800 5700
+F 0 "#PWR020" H 4800 5450 50  0001 C CNN
+F 1 "GND" H 4805 5527 50  0000 C CNN
+F 2 "" H 4800 5700 50  0001 C CNN
+F 3 "" H 4800 5700 50  0001 C CNN
+	1    4800 5700
+	1    0    0    -1
+$EndComp
+Wire Wire Line
+	4800 5600 4800 5700
+Connection ~ 4800 5600
+Wire Wire Line
+	4750 5600 4800 5600
+Wire Wire Line
+	4800 5400 4800 5600
+Connection ~ 4800 5400
+Wire Wire Line
+	4750 5400 4800 5400
+Wire Wire Line
+	4800 5300 4800 5400
+Connection ~ 4800 5300
+Wire Wire Line
+	4750 5300 4800 5300
+Wire Wire Line
+	4800 5200 4800 5300
+Wire Wire Line
+	4750 5200 4800 5200
+Wire Wire Line
+	4750 4400 5200 4400
+Text Label 5200 4400 2    50   ~ 0
+ESP_TX
+Wire Wire Line
+	4750 4300 5200 4300
+Text Label 5200 4300 2    50   ~ 0
+ESP_RX
 $Comp
 L PlayboardLib:ESP32-WROVER-I U4
@@
 	1    0    0    -1
 $EndComp
-NoConn ~ 4750 4900
-NoConn ~ 4750 5000
-NoConn ~ 3550 5900
-Text Label 3100 4600 0    50   ~ 0
-GPIO0
-Wire Wire Line
-	4750 4800 5200 4800
-Wire Wire Line
-	4750 4600 5200 4600
-Text Label 5200 4800 2    50   ~ 0
-IR_SEND
-Text Label 5200 4600 2    50   ~ 0
-IR_RECV
-$Comp
-L power:GND #PWR020
-U 1 1 61CED5C0
-P 4800 5700
-F 0 "#PWR020" H 4800 5450 50  0001 C CNN
-F 1 "GND" H 4805 5527 50  0000 C CNN
-F 2 "" H 4800 5700 50  0001 C CNN
-F 3 "" H 4800 5700 50  0001 C CNN
-	1    4800 5700
-	1    0    0    -1
-$EndComp
-Wire Wire Line
-	4800 5600 4800 5700
-Connection ~ 4800 5600
-Wire Wire Line
-	4750 5600 4800 5600
-Wire Wire Line
-	4800 5400 4800 5600
-Connection ~ 4800 5400
-Wire Wire Line
-	4750 5400 4800 5400
-Wire Wire Line
-	4800 5300 4800 5400
-Connection ~ 4800 5300
-Wire Wire Line
-	4750 5300 4800 5300
-Wire Wire Line
-	4800 5200 4800 5300
-Wire Wire Line
-	4750 5200 4800 5200
-Wire Wire Line
-	4750 4400 5200 4400
-Text Label 5200 4400 2    50   ~ 0
-ESP_TX
-Wire Wire Line
-	4750 4300 5200 4300
-Text Label 5200 4300 2    50   ~ 0
-ESP_RX
 $EndSCHEMATC
